Commit message: replace file:// with package://

File: denso_robot_descriptions/robots/cobotta/urdf/denso_robot_kinematics.xacro (robot description, xacro)
@@ -11,5 +11,5 @@
 				<origin rpy="0 0 0" xyz="0 0 0"/>
 				<geometry>
-					<mesh filename="file:///$(find denso_robot_descriptions)/robots/$(arg model)/meshes/base_link.dae" scale="1 1 1"/>
+					<mesh filename="package://denso_robot_descriptions/robots/$(arg model)/meshes/base_link.dae" scale="1 1 1"/>
 				</geometry>
 			</visual>
@@ -17,5 +17,5 @@
 				<origin rpy="0 0 0" xyz="0 0 0"/>
 				<geometry>
-					<mesh filename="file:///$(find denso_robot_descriptions)/robots/$(arg model)/meshes/base_link.dae" scale="1 1 1"/>
+					<mesh filename="package://denso_robot_descriptions/robots/$(arg model)/meshes/base_link.dae" scale="1 1 1"/>
 				</geometry>
 			</collision>
@@ -30,5 +30,5 @@
 				<origin rpy="0 0 0" xyz="0 0 0"/>
 				<geometry>
-					<mesh filename="file:///$(find denso_robot_descriptions)/robots/$(arg model)/meshes/J1.dae" scale="1 1 1"/>
+					<mesh filename="package://denso_robot_descriptions/robots/$(arg model)/meshes/J1.dae" scale="1 1 1"/>
 				</geometry>
 			</visual>
@@ -36,5 +36,5 @@
 				<origin rpy="0 0 0" xyz="0 0 0"/>
 				<geometry>
-					<mesh filename="file:///$(find denso_robot_descriptions)/robots/$(arg model)/meshes/J1.dae" scale="1 1 1"/>
+					<mesh filename="package://denso_robot_descriptions/robots/$(arg model)/meshes/J1.dae" scale="1 1 1"/>
 				</geometry>
 			</collision>
@@ -57,5 +57,5 @@
 				<origin rpy="0 0 0" xyz="0 0 0"/>
 				<geometry>
-					<mesh filename="file:///$(find denso_robot_descriptions)/robots/$(arg model)/meshes/J2.dae" scale="1 1 1"/>
+					<mesh filename="package://denso_robot_descriptions/robots/$(arg model)/meshes/J2.dae" scale="1 1 1"/>
 				</geometry>
 			</visual>
@@ -63,5 +63,5 @@
 				<origin rpy="0 0 0" xyz="0 0 0"/>
 				<geometry>
-					<mesh filename="file:///$(find denso_robot_descriptions)/robots/$(arg model)/meshes/J2.dae" scale="1 1 1"/>
+					<mesh filename="package://denso_robot_descriptions/robots/$(arg model)/meshes/J2.dae" scale="1 1 1"/>
 				</geometry>
 			</collision>
@@ -84,5 +84,5 @@
 				<origin rpy="0 0 0" xyz="0 0 0"/>
 				<geometry>
-					<mesh filename="file:///$(find denso_robot_descriptions)/robots/$(arg model)/meshes/J3.dae" scale="1 1 1"/>
+					<mesh filename="package://denso_robot_descriptions/robots/$(arg model)/meshes/J3.dae" scale="1 1 1"/>
 				</geometry>
 			</visual>
@@ -90,5 +90,5 @@
 				<origin rpy="0 0 0" xyz="0 0 0"/>
 				<geometry>
-					<mesh filename="file:///$(find denso_robot_descriptions)/robots/$(arg model)/meshes/J3.dae" scale="1 1 1"/>
+					<mesh filename="package://denso_robot_descriptions/robots/$(arg model)/meshes/J3.dae" scale="1 1 1"/>
 				</geometry>
 			</collision>
@@ -111,5 +111,5 @@
 				<origin rpy="0 0 0" xyz="0 0 0"/>
 				<geometry>
-					<mesh filename="file:///$(find denso_robot_descriptions)/robots/$(arg model)/meshes/J4.dae" scale="1 1 1"/>
+					<mesh filename="package://denso_robot_descriptions/robots/$(arg model)/meshes/J4.dae" scale="1 1 1"/>
 				</geometry>
 			</visual>
@@ -117,5 +117,5 @@
 				<origin rpy="0 0 0" xyz="0 0 0"/>
 				<geometry>
-					<mesh filename="file:///$(find denso_robot_descriptions)/robots/$(arg model)/meshes/J4.dae" scale="1 1 1"/>
+					<mesh filename="package://denso_robot_descriptions/robots/$(arg model)/meshes/J4.dae" scale="1 1 1"/>
 				</geometry>
 			</collision>
@@ -138,5 +138,5 @@
 				<origin rpy="0 0 0" xyz="0 0 0"/>
 				<geometry>
-					<mesh filename="file:///$(find denso_robot_descriptions)/robots/$(arg model)/meshes/J5.dae" scale="1 1 1"/>
+					<mesh filename="package://denso_robot_descriptions/robots/$(arg model)/meshes/J5.dae" scale="1 1 1"/>
 				</geometry>
 			</visual>
@@ -144,5 +144,5 @@
 				<origin rpy="0 0 0" xyz="0 0 0"/>
 				<geometry>
-					<mesh filename="file:///$(find denso_robot_descriptions)/robots/$(arg model)/meshes/J5.dae" scale="1 1 1"/>
+					<mesh filename="package://denso_robot_descriptions/robots/$(arg model)/meshes/J5.dae" scale="1 1 1"/>
 				</geometry>
 			</collision>
@@ -165,5 +165,5 @@
 				<origin rpy="0 0 0" xyz="0 0 0"/>
 				<geometry>
-					<mesh filename="file:///$(find denso_robot_descriptions)/robots/$(arg model)/meshes/J6.dae" scale="1 1 1"/>
+					<mesh filename="package://denso_robot_descriptions/robots/$(arg model)/meshes/J6.dae" scale="1 1 1"/>
 				</geometry>
 			</visual>
@@ -171,5 +171,5 @@
 				<origin rpy="0 0 0" xyz="0 0 0"/>
 				<geometry>
-					<mesh filename="file:///$(find denso_robot_descriptions)/robots/$(arg model)/meshes/J6.dae" scale="1 1 1"/>
+					<mesh filename="package://denso_robot_descriptions/robots/$(arg model)/meshes/J6.dae" scale="1 1 1"/>
 				</geometry>
 			</collision>

File: denso_robot_descriptions/robots/cvrb0609/urdf/denso_robot_kinematics.xacro (robot description, xacro)
@@ -11,5 +11,5 @@
 				<origin rpy="0 0 0" xyz="0 0 0"/>
 				<geometry>
-					<mesh filename="file:///$(find denso_robot_descriptions)/robots/$(arg model)/meshes/base_link.dae" scale="1 1 1"/>
+					<mesh filename="package://denso_robot_descriptions/robots/$(arg model)/meshes/base_link.dae" scale="1 1 1"/>
 				</geometry>
 			</visual>
@@ -17,5 +17,5 @@
 				<origin rpy="0 0 0" xyz="0 0 0"/>
 				<geometry>
-					<mesh filename="file:///$(find denso_robot_descriptions)/robots/$(arg model)/meshes/base_link.dae" scale="1 1 1"/>
+					<mesh filename="package://denso_robot_descriptions/robots/$(arg model)/meshes/base_link.dae" scale="1 1 1"/>
 				</geometry>
 			</collision>
@@ -30,5 +30,5 @@
 				<origin rpy="0 0 0" xyz="0 0 0"/>
 				<geometry>
-					<mesh filename="file:///$(find denso_robot_descriptions)/robots/$(arg model)/meshes/J1.dae" scale="1 1 1"/>
+					<mesh filename="package://denso_robot_descriptions/robots/$(arg model)/meshes/J1.dae" scale="1 1 1"/>
 				</geometry>
 			</visual>
@@ -36,5 +36,5 @@
 				<origin rpy="0 0 0" xyz="0 0 0"/>
 				<geometry>
-					<mesh filename="file:///$(find denso_robot_descriptions)/robots/$(arg model)/meshes/J1.dae" scale="1 1 1"/>
+					<mesh filename="package://denso_robot_descriptions/robots/$(arg model)/meshes/J1.dae" scale="1 1 1"/>
 				</geometry>
 			</collision>
@@ -57,5 +57,5 @@
 				<origin rpy="0 0 0" xyz="0 0 0"/>
 				<geometry>
-					<mesh filename="file:///$(find denso_robot_descriptions)/robots/$(arg model)/meshes/J2.dae" scale="1 1 1"/>
+					<mesh filename="package://denso_robot_descriptions/robots/$(arg model)/meshes/J2.dae" scale="1 1 1"/>
 				</geometry>
 			</visual>
@@ -63,5 +63,5 @@
 				<origin rpy="0 0 0" xyz="0 0 0"/>
 				<geometry>
-					<mesh filename="file:///$(find denso_robot_descriptions)/robots/$(arg model)/meshes/J2.dae" scale="1 1 1"/>
+					<mesh filename="package://denso_robot_descriptions/robots/$(arg model)/meshes/J2.dae" scale="1 1 1"/>
 				</geometry>
 			</collision>
@@ -84,5 +84,5 @@
 				<origin rpy="0 0 0" xyz="0 0 0"/>
 				<geometry>
-					<mesh filename="file:///$(find denso_robot_descriptions)/robots/$(arg model)/meshes/J3.dae" scale="1 1 1"/>
+					<mesh filename="package://denso_robot_descriptions/robots/$(arg model)/meshes/J3.dae" scale="1 1 1"/>
 				</geometry>
 			</visual>
@@ -90,5 +90,5 @@
 				<origin rpy="0 0 0" xyz="0 0 0"/>
 				<geometry>
-					<mesh filename="file:///$(find denso_robot_descriptions)/robots/$(arg model)/meshes/J3.dae" scale="1 1 1"/>
+					<mesh filename="package://denso_robot_descriptions/robots/$(arg model)/meshes/J3.dae" scale="1 1 1"/>
 				</geometry>
 			</collision>
@@ -111,5 +111,5 @@
 				<origin rpy="0 0 0" xyz="0 0 0"/>
 				<geometry>
-					<mesh filename="file:///$(find denso_robot_descriptions)/robots/$(arg model)/meshes/J4.dae" scale="1 1 1"/>
+					<mesh filename="package://denso_robot_descriptions/robots/$(arg model)/meshes/J4.dae" scale="1 1 1"/>
 				</geometry>
 			</visual>
@@ -117,5 +117,5 @@
 				<origin rpy="0 0 0" xyz="0 0 0"/>
 				<geometry>
-					<mesh filename="file:///$(find denso_robot_descriptions)/robots/$(arg model)/meshes/J4.dae" scale="1 1 1"/>
+					<mesh filename="package://denso_robot_descriptions/robots/$(arg model)/meshes/J4.dae" scale="1 1 1"/>
 				</geometry>
 			</collision>
@@ -138,5 +138,5 @@
 				<origin rpy="0 0 0" xyz="0 0 0"/>
 				<geometry>
-					<mesh filename="file:///$(find denso_robot_descriptions)/robots/$(arg model)/meshes/J5.dae" scale="1 1 1"/>
+					<mesh filename="package://denso_robot_descriptions/robots/$(arg model)/meshes/J5.dae" scale="1 1 1"/>
 				</geometry>
 			</visual>
@@ -144,5 +144,5 @@
 				<origin rpy="0 0 0" xyz="0 0 0"/>
 				<geometry>
-					<mesh filename="file:///$(find denso_robot_descriptions)/robots/$(arg model)/meshes/J5.dae" scale="1 1 1"/>
+					<mesh filename="package://denso_robot_descriptions/robots/$(arg model)/meshes/J5.dae" scale="1 1 1"/>
 				</geometry>
 			</collision>
@@ -165,5 +165,5 @@
 				<origin rpy="0 0 0" xyz="0 0 0"/>
 				<geometry>
-					<mesh filename="file:///$(find denso_robot_descriptions)/robots/$(arg model)/meshes/J6.dae" scale="1 1 1"/>
+					<mesh filename="package://denso_robot_descriptions/robots/$(arg model)/meshes/J6.dae" scale="1 1 1"/>
 				</geometry>
 			</visual>
@@ -171,5 +171,5 @@
 				<origin rpy="0 0 0" xyz="0 0 0"/>
 				<geometry>
-					<mesh filename="file:///$(find denso_robot_descriptions)/robots/$(arg model)/meshes/J6.dae" scale="1 1 1"/>
+					<mesh filename="package://denso_robot_descriptions/robots/$(arg model)/meshes/J6.dae" scale="1 1 1"/>
 				</geometry>
 			</collision>

File: denso_robot_descriptions/robots/hsr065a1_n32/urdf/denso_robot_kinematics.xacro (robot description, xacro)
@@ -11,5 +11,5 @@
 				<origin rpy="0 0 0" xyz="0 0 0"/>
 				<geometry>
-					<mesh filename="file:///$(find denso_robot_descriptions)/robots/$(arg model)/meshes/base_link.dae" scale="1 1 1"/>
+					<mesh filename="package://denso_robot_descriptions/robots/$(arg model)/meshes/base_link.dae" scale="1 1 1"/>
 				</geometry>
 			</visual>
@@ -17,5 +17,5 @@
 				<origin rpy="0 0 0" xyz="0 0 0"/>
 				<geometry>
-					<mesh filename="file:///$(find denso_robot_descriptions)/robots/$(arg model)/meshes/base_link.dae" scale="1 1 1"/>
+					<mesh filename="package://denso_robot_descriptions/robots/$(arg model)/meshes/base_link.dae" scale="1 1 1"/>
 				</geometry>
 			</collision>
@@ -30,5 +30,5 @@
 				<origin rpy="0 0 0" xyz="0 0 0"/>
 				<geometry>
-					<mesh filename="file:///$(find denso_robot_descriptions)/robots/$(arg model)/meshes/J1.dae" scale="1 1 1"/>
+					<mesh filename="package://denso_robot_descriptions/robots/$(arg model)/meshes/J1.dae" scale="1 1 1"/>
 				</geometry>
 			</visual>
@@ -36,5 +36,5 @@
 				<origin rpy="0 0 0" xyz="0 0 0"/>
 				<geometry>
-					<mesh filename="file:///$(find denso_robot_descriptions)/robots/$(arg model)/meshes/J1.dae" scale="1 1 1"/>
+					<mesh filename="package://denso_robot_descriptions/robots/$(arg model)/meshes/J1.dae" scale="1 1 1"/>
 				</geometry>
 			</collision>
@@ -57,5 +57,5 @@
 				<origin rpy="0 0 0" xyz="0 0 0"/>
 				<geometry>
-					<mesh filename="file:///$(find denso_robot_descriptions)/robots/$(arg model)/meshes/J2.dae" scale="1 1 1"/>
+					<mesh filename="package://denso_robot_descriptions/robots/$(arg model)/meshes/J2.dae" scale="1 1 1"/>
 				</geometry>
 			</visual>
@@ -63,5 +63,5 @@
 				<origin rpy="0 0 0" xyz="0 0 0"/>
 				<geometry>
-					<mesh filename="file:///$(find denso_robot_descriptions)/robots/$(arg model)/meshes/J2.dae" scale="1 1 1"/>
+					<mesh filename="package://denso_robot_descriptions/robots/$(arg model)/meshes/J2.dae" scale="1 1 1"/>
 				</geometry>
 			</collision>
@@ -84,5 +84,5 @@
 				<origin rpy="0 0 0" xyz="0 0 0"/>
 				<geometry>
-					<mesh filename="file:///$(find denso_robot_descriptions)/robots/$(arg model)/meshes/J3.dae" scale="1 1 1"/>
+					<mesh filename="package://denso_robot_descriptions/robots/$(arg model)/meshes/J3.dae" scale="1 1 1"/>
 				</geometry>
 			</visual>
@@ -90,5 +90,5 @@
 				<origin rpy="0 0 0" xyz="0 0 0"/>
 				<geometry>
-					<mesh filename="file:///$(find denso_robot_descriptions)/robots/$(arg model)/meshes/J3.dae" scale="1 1 1"/>
+					<mesh filename="package://denso_robot_descriptions/robots/$(arg model)/meshes/J3.dae" scale="1 1 1"/>
 				</geometry>
 			</collision>
@@ -111,5 +111,5 @@
 				<origin rpy="0 0 0" xyz="0 0 0"/>
 				<geometry>
-					<mesh filename="file:///$(find denso_robot_descriptions)/robots/$(arg model)/meshes/J4.dae" scale="1 1 1"/>
+					<mesh filename="package://denso_robot_descriptions/robots/$(arg model)/meshes/J4.dae" scale="1 1 1"/>
 				</geometry>
 			</visual>
@@ -117,5 +117,5 @@
 				<origin rpy="0 0 0" xyz="0 0 0"/>
 				<geometry>
-					<mesh filename="file:///$(find denso_robot_descriptions)/robots/$(arg model)/meshes/J4.dae" scale="1 1 1"/>
+					<mesh filename="package://denso_robot_descriptions/robots/$(arg model)/meshes/J4.dae" scale="1 1 1"/>
 				</geometry>
 			</collision>

File: denso_robot_descriptions/robots/vs060/urdf/denso_robot_kinematics.xacro (robot description, xacro)
@@ -11,5 +11,5 @@
 				<origin rpy="0 0 0" xyz="0 0 0"/>
 				<geometry>
-					<mesh filename="file:///$(find denso_robot_descriptions)/robots/$(arg model)/meshes/base_link.dae" scale="1 1 1"/>
+					<mesh filename="package://denso_robot_descriptions/robots/$(arg model)/meshes/base_link.dae" scale="1 1 1"/>
 				</geometry>
 			</visual>
@@ -17,5 +17,5 @@
 				<origin rpy="0 0 0" xyz="0 0 0"/>
 				<geometry>
-					<mesh filename="file:///$(find denso_robot_descriptions)/robots/$(arg model)/meshes/base_link.dae" scale="1 1 1"/>
+					<mesh filename="package://denso_robot_descriptions/robots/$(arg model)/meshes/base_link.dae" scale="1 1 1"/>
 				</geometry>
 			</collision>
@@ -30,5 +30,5 @@
 				<origin rpy="0 0 0" xyz="0 0 0"/>
 				<geometry>
-					<mesh filename="file:///$(find denso_robot_descriptions)/robots/$(arg model)/meshes/J1.dae" scale="1 1 1"/>
+					<mesh filename="package://denso_robot_descriptions/robots/$(arg model)/meshes/J1.dae" scale="1 1 1"/>
 				</geometry>
 			</visual>
@@ -36,5 +36,5 @@
 				<origin rpy="0 0 0" xyz="0 0 0"/>
 				<geometry>
-					<mesh filename="file:///$(find denso_robot_descriptions)/robots/$(arg model)/meshes/J1.dae" scale="1 1 1"/>
+					<mesh filename="package://denso_robot_descriptions/robots/$(arg model)/meshes/J1.dae" scale="1 1 1"/>
 				</geometry>
 			</collision>
@@ -57,5 +57,5 @@
 				<origin rpy="0 0 0" xyz="0 0 0"/>
 				<geometry>
-					<mesh filename="file:///$(find denso_robot_descriptions)/robots/$(arg model)/meshes/J2.dae" scale="1 1 1"/>
+					<mesh filename="package://denso_robot_descriptions/robots/$(arg model)/meshes/J2.dae" scale="1 1 1"/>
 				</geometry>
 			</visual>
@@ -63,5 +63,5 @@
 				<origin rpy="0 0 0" xyz="0 0 0"/>
 				<geometry>
-					<mesh filename="file:///$(find denso_robot_descriptions)/robots/$(arg model)/meshes/J2.dae" scale="1 1 1"/>
+					<mesh filename="package://denso_robot_descriptions/robots/$(arg model)/meshes/J2.dae" scale="1 1 1"/>
 				</geometry>
 			</collision>
@@ -84,5 +84,5 @@
 				<origin rpy="0 0 0" xyz="0 0 0"/>
 				<geometry>
-					<mesh filename="file:///$(find denso_robot_descriptions)/robots/$(arg model)/meshes/J3.dae" scale="1 1 1"/>
+					<mesh filename="package://denso_robot_descriptions/robots/$(arg model)/meshes/J3.dae" scale="1 1 1"/>
 				</geometry>
 			</visual>
@@ -90,5 +90,5 @@
 				<origin rpy="0 0 0" xyz="0 0 0"/>
 				<geometry>
-					<mesh filename="file:///$(find denso_robot_descriptions)/robots/$(arg model)/meshes/J3.dae" scale="1 1 1"/>
+					<mesh filename="package://denso_robot_descriptions/robots/$(arg model)/meshes/J3.dae" scale="1 1 1"/>
 				</geometry>
 			</collision>
@@ -111,5 +111,5 @@
 				<origin rpy="0 0 0" xyz="0 0 0"/>
 				<geometry>
-					<mesh filename="file:///$(find denso_robot_descriptions)/robots/$(arg model)/meshes/J4.dae" scale="1 1 1"/>
+					<mesh filename="package://denso_robot_descriptions/robots/$(arg model)/meshes/J4.dae" scale="1 1 1"/>
 				</geometry>
 			</visual>
@@ -117,5 +117,5 @@
 				<origin rpy="0 0 0" xyz="0 0 0"/>
 				<geometry>
-					<mesh filename="file:///$(find denso_robot_descriptions)/robots/$(arg model)/meshes/J4.dae" scale="1 1 1"/>
+					<mesh filename="package://denso_robot_descriptions/robots/$(arg model)/meshes/J4.dae" scale="1 1 1"/>
 				</geometry>
 			</collision>
@@ -138,5 +138,5 @@
 				<origin rpy="0 0 0" xyz="0 0 0"/>
 				<geometry>
-					<mesh filename="file:///$(find denso_robot_descriptions)/robots/$(arg model)/meshes/J5.dae" scale="1 1 1"/>
+					<mesh filename="package://denso_robot_descriptions/robots/$(arg model)/meshes/J5.dae" scale="1 1 1"/>
 				</geometry>
 			</visual>
@@ -144,5 +144,5 @@
 				<origin rpy="0 0 0" xyz="0 0 0"/>
 				<geometry>
-					<mesh filename="file:///$(find denso_robot_descriptions)/robots/$(arg model)/meshes/J5.dae" scale="1 1 1"/>
+					<mesh filename="package://denso_robot_descriptions/robots/$(arg model)/meshes/J5.dae" scale="1 1 1"/>
 				</geometry>
 			</collision>
@@ -165,5 +165,5 @@
 				<origin rpy="0 0 0" xyz="0 0 0"/>
 				<geometry>
-					<mesh filename="file:///$(find denso_robot_descriptions)/robots/$(arg model)/meshes/J6.dae" scale="1 1 1"/>
+					<mesh filename="package://denso_robot_descriptions/robots/$(arg model)/meshes/J6.dae" scale="1 1 1"/>
 				</geometry>
 			</visual>
@@ -171,5 +171,5 @@
 				<origin rpy="0 0 0" xyz="0 0 0"/>
 				<geometry>
-					<mesh filename="file:///$(find denso_robot_descriptions)/robots/$(arg model)/meshes/J6.dae" scale="1 1 1"/>
+					<mesh filename="package://denso_robot_descriptions/robots/$(arg model)/meshes/J6.dae" scale="1 1 1"/>
 				</geometry>
 			</collision>
