Commit message: remove /

File: cvrb0609_description/urdf/cvrb0609.urdf.xacro (robot description, xacro)
@@ -23,11 +23,11 @@
       <origin rpy="0 0 0" xyz="0 0 0"/>
       <geometry>
-        <mesh filename="package://cvrb0609_description/meshes//base_link.dae" scale="1 1 1"/>
-      </geometry>
-    </visual>
-    <collision>
-      <origin rpy="0 0 0" xyz="0 0 0"/>
-      <geometry>
-        <mesh filename="package://cvrb0609_description/meshes//base_link.dae" scale="1 1 1"/>
+        <mesh filename="package://cvrb0609_description/meshes/base_link.dae" scale="1 1 1"/>
+      </geometry>
+    </visual>
+    <collision>
+      <origin rpy="0 0 0" xyz="0 0 0"/>
+      <geometry>
+        <mesh filename="package://cvrb0609_description/meshes/base_link.dae" scale="1 1 1"/>
       </geometry>
     </collision>
@@ -42,11 +42,11 @@
       <origin rpy="0 0 0" xyz="0 0 0"/>
       <geometry>
-        <mesh filename="package://cvrb0609_description/meshes//J1.dae" scale="1 1 1"/>
-      </geometry>
-    </visual>
-    <collision>
-      <origin rpy="0 0 0" xyz="0 0 0"/>
-      <geometry>
-        <mesh filename="package://cvrb0609_description/meshes//J1.dae" scale="1 1 1"/>
+        <mesh filename="package://cvrb0609_description/meshes/J1.dae" scale="1 1 1"/>
+      </geometry>
+    </visual>
+    <collision>
+      <origin rpy="0 0 0" xyz="0 0 0"/>
+      <geometry>
+        <mesh filename="package://cvrb0609_description/meshes/J1.dae" scale="1 1 1"/>
       </geometry>
     </collision>
@@ -69,11 +69,11 @@
       <origin rpy="0 0 0" xyz="0 0 0"/>
       <geometry>
-        <mesh filename="package://cvrb0609_description/meshes//J2.dae" scale="1 1 1"/>
-      </geometry>
-    </visual>
-    <collision>
-      <origin rpy="0 0 0" xyz="0 0 0"/>
-      <geometry>
-        <mesh filename="package://cvrb0609_description/meshes//J2.dae" scale="1 1 1"/>
+        <mesh filename="package://cvrb0609_description/meshes/J2.dae" scale="1 1 1"/>
+      </geometry>
+    </visual>
+    <collision>
+      <origin rpy="0 0 0" xyz="0 0 0"/>
+      <geometry>
+        <mesh filename="package://cvrb0609_description/meshes/J2.dae" scale="1 1 1"/>
       </geometry>
     </collision>
@@ -96,11 +96,11 @@
       <origin rpy="0 0 0" xyz="0 0 0"/>
       <geometry>
-        <mesh filename="package://cvrb0609_description/meshes//J3.dae" scale="1 1 1"/>
-      </geometry>
-    </visual>
-    <collision>
-      <origin rpy="0 0 0" xyz="0 0 0"/>
-      <geometry>
-        <mesh filename="package://cvrb0609_description/meshes//J3.dae" scale="1 1 1"/>
+        <mesh filename="package://cvrb0609_description/meshes/J3.dae" scale="1 1 1"/>
+      </geometry>
+    </visual>
+    <collision>
+      <origin rpy="0 0 0" xyz="0 0 0"/>
+      <geometry>
+        <mesh filename="package://cvrb0609_description/meshes/J3.dae" scale="1 1 1"/>
       </geometry>
     </collision>
@@ -123,11 +123,11 @@
       <origin rpy="0 0 0" xyz="0 0 0"/>
       <geometry>
-        <mesh filename="package://cvrb0609_description/meshes//J4.dae" scale="1 1 1"/>
-      </geometry>
-    </visual>
-    <collision>
-      <origin rpy="0 0 0" xyz="0 0 0"/>
-      <geometry>
-        <mesh filename="package://cvrb0609_description/meshes//J4.dae" scale="1 1 1"/>
+        <mesh filename="package://cvrb0609_description/meshes/J4.dae" scale="1 1 1"/>
+      </geometry>
+    </visual>
+    <collision>
+      <origin rpy="0 0 0" xyz="0 0 0"/>
+      <geometry>
+        <mesh filename="package://cvrb0609_description/meshes/J4.dae" scale="1 1 1"/>
       </geometry>
     </collision>
@@ -150,11 +150,11 @@
       <origin rpy="0 0 0" xyz="0 0 0"/>
       <geometry>
-        <mesh filename="package://cvrb0609_description/meshes//J5.dae" scale="1 1 1"/>
-      </geometry>
-    </visual>
-    <collision>
-      <origin rpy="0 0 0" xyz="0 0 0"/>
-      <geometry>
-        <mesh filename="package://cvrb0609_description/meshes//J5.dae" scale="1 1 1"/>
+        <mesh filename="package://cvrb0609_description/meshes/J5.dae" scale="1 1 1"/>
+      </geometry>
+    </visual>
+    <collision>
+      <origin rpy="0 0 0" xyz="0 0 0"/>
+      <geometry>
+        <mesh filename="package://cvrb0609_description/meshes/J5.dae" scale="1 1 1"/>
       </geometry>
     </collision>
@@ -177,11 +177,11 @@
       <origin rpy="0 0 0" xyz="0 0 0"/>
       <geometry>
-        <mesh filename="package://cvrb0609_description/meshes//J6.dae" scale="1 1 1"/>
-      </geometry>
-    </visual>
-    <collision>
-      <origin rpy="0 0 0" xyz="0 0 0"/>
-      <geometry>
-        <mesh filename="package://cvrb0609_description/meshes//J6.dae" scale="1 1 1"/>
+        <mesh filename="package://cvrb0609_description/meshes/J6.dae" scale="1 1 1"/>
+      </geometry>
+    </visual>
+    <collision>
+      <origin rpy="0 0 0" xyz="0 0 0"/>
+      <geometry>
+        <mesh filename="package://cvrb0609_description/meshes/J6.dae" scale="1 1 1"/>
       </geometry>
     </collision>

Commit message: remove  scale="1 1 1"

File: cvrb0609_description/urdf/cvrb0609.urdf.xacro (robot description, xacro)
@@ -23,11 +23,11 @@
       <origin rpy="0 0 0" xyz="0 0 0"/>
       <geometry>
-        <mesh filename="package://cvrb0609_description/meshes/base_link.dae" scale="1 1 1"/>
-      </geometry>
-    </visual>
-    <collision>
-      <origin rpy="0 0 0" xyz="0 0 0"/>
-      <geometry>
-        <mesh filename="package://cvrb0609_description/meshes/base_link.dae" scale="1 1 1"/>
+        <mesh filename="package://cvrb0609_description/meshes/base_link.dae"/>
+      </geometry>
+    </visual>
+    <collision>
+      <origin rpy="0 0 0" xyz="0 0 0"/>
+      <geometry>
+        <mesh filename="package://cvrb0609_description/meshes/base_link.dae"/>
       </geometry>
     </collision>
@@ -42,11 +42,11 @@
       <origin rpy="0 0 0" xyz="0 0 0"/>
       <geometry>
-        <mesh filename="package://cvrb0609_description/meshes/J1.dae" scale="1 1 1"/>
-      </geometry>
-    </visual>
-    <collision>
-      <origin rpy="0 0 0" xyz="0 0 0"/>
-      <geometry>
-        <mesh filename="package://cvrb0609_description/meshes/J1.dae" scale="1 1 1"/>
+        <mesh filename="package://cvrb0609_description/meshes/J1.dae"/>
+      </geometry>
+    </visual>
+    <collision>
+      <origin rpy="0 0 0" xyz="0 0 0"/>
+      <geometry>
+        <mesh filename="package://cvrb0609_description/meshes/J1.dae"/>
       </geometry>
     </collision>
@@ -69,11 +69,11 @@
       <origin rpy="0 0 0" xyz="0 0 0"/>
       <geometry>
-        <mesh filename="package://cvrb0609_description/meshes/J2.dae" scale="1 1 1"/>
-      </geometry>
-    </visual>
-    <collision>
-      <origin rpy="0 0 0" xyz="0 0 0"/>
-      <geometry>
-        <mesh filename="package://cvrb0609_description/meshes/J2.dae" scale="1 1 1"/>
+        <mesh filename="package://cvrb0609_description/meshes/J2.dae"/>
+      </geometry>
+    </visual>
+    <collision>
+      <origin rpy="0 0 0" xyz="0 0 0"/>
+      <geometry>
+        <mesh filename="package://cvrb0609_description/meshes/J2.dae"/>
       </geometry>
     </collision>
@@ -96,11 +96,11 @@
       <origin rpy="0 0 0" xyz="0 0 0"/>
       <geometry>
-        <mesh filename="package://cvrb0609_description/meshes/J3.dae" scale="1 1 1"/>
-      </geometry>
-    </visual>
-    <collision>
-      <origin rpy="0 0 0" xyz="0 0 0"/>
-      <geometry>
-        <mesh filename="package://cvrb0609_description/meshes/J3.dae" scale="1 1 1"/>
+        <mesh filename="package://cvrb0609_description/meshes/J3.dae"/>
+      </geometry>
+    </visual>
+    <collision>
+      <origin rpy="0 0 0" xyz="0 0 0"/>
+      <geometry>
+        <mesh filename="package://cvrb0609_description/meshes/J3.dae"/>
       </geometry>
     </collision>
@@ -123,11 +123,11 @@
       <origin rpy="0 0 0" xyz="0 0 0"/>
       <geometry>
-        <mesh filename="package://cvrb0609_description/meshes/J4.dae" scale="1 1 1"/>
-      </geometry>
-    </visual>
-    <collision>
-      <origin rpy="0 0 0" xyz="0 0 0"/>
-      <geometry>
-        <mesh filename="package://cvrb0609_description/meshes/J4.dae" scale="1 1 1"/>
+        <mesh filename="package://cvrb0609_description/meshes/J4.dae"/>
+      </geometry>
+    </visual>
+    <collision>
+      <origin rpy="0 0 0" xyz="0 0 0"/>
+      <geometry>
+        <mesh filename="package://cvrb0609_description/meshes/J4.dae"/>
       </geometry>
     </collision>
@@ -150,11 +150,11 @@
       <origin rpy="0 0 0" xyz="0 0 0"/>
       <geometry>
-        <mesh filename="package://cvrb0609_description/meshes/J5.dae" scale="1 1 1"/>
-      </geometry>
-    </visual>
-    <collision>
-      <origin rpy="0 0 0" xyz="0 0 0"/>
-      <geometry>
-        <mesh filename="package://cvrb0609_description/meshes/J5.dae" scale="1 1 1"/>
+        <mesh filename="package://cvrb0609_description/meshes/J5.dae"/>
+      </geometry>
+    </visual>
+    <collision>
+      <origin rpy="0 0 0" xyz="0 0 0"/>
+      <geometry>
+        <mesh filename="package://cvrb0609_description/meshes/J5.dae"/>
       </geometry>
     </collision>
@@ -177,11 +177,11 @@
       <origin rpy="0 0 0" xyz="0 0 0"/>
       <geometry>
-        <mesh filename="package://cvrb0609_description/meshes/J6.dae" scale="1 1 1"/>
-      </geometry>
-    </visual>
-    <collision>
-      <origin rpy="0 0 0" xyz="0 0 0"/>
-      <geometry>
-        <mesh filename="package://cvrb0609_description/meshes/J6.dae" scale="1 1 1"/>
+        <mesh filename="package://cvrb0609_description/meshes/J6.dae"/>
+      </geometry>
+    </visual>
+    <collision>
+      <origin rpy="0 0 0" xyz="0 0 0"/>
+      <geometry>
+        <mesh filename="package://cvrb0609_description/meshes/J6.dae"/>
       </geometry>
     </collision>
